File: Schematics/CargaElectronica.kicad_sch (KiCad schematic)
At the start: 40 parts, among them J1 Voltage_test, J2 Voltage_IN, Q1 IRFP460, SW1 Rotary_Encoder_Switch, SW2 Btn.OK, SW3 Btn.BCK, U1 TL072, U2 Pantalla_LCD_16x2_i2c, U3 LM35-LP, U4 TL431DBZ

Commit message: Imagen y documentos de la PCB
Other:
- company: (none) -> Laboratorio Gluon
- title: (none) -> ArduDCLoad

Commit message: Updated schematic, did not update with last commit
Parts:
- added D2: D_Schottky, Diode_SMD:D_SOD-323_HandSoldering, symbol Device:D_Schottky
- added HS1: Heatsink, symbol Mechanical:Heatsink
- added J3: FAN_OUTPUT, Connector_PinHeader_2.54mm:PinHeader_1x02_P2.54mm_Vertical, symbol Connector:Screw_Terminal_01x02
- added Q2: Q_NMOS_GSD, Package_TO_SOT_SMD:SOT-23, symbol Device:Q_NMOS_GSD
- added R24: 1Meg, Resistor_SMD:R_1206_3216Metric_Pad1.30x1.75mm_HandSolder, symbol Device:R
- added R3: 330, Resistor_SMD:R_1206_3216Metric_Pad1.30x1.75mm_HandSolder, symbol Device:R
- added TP5: FanCtrl, TestPoint:TestPoint_Pad_D2.0mm, symbol Connector:TestPoint
Connections:
- net GND: now also Q2.2 (S), R24.1
- net V_IN: now also D2.1 (K), J3.1 (Pin_1)
- net FAN_CONTROL: now reaches A1.8 (D5)
- net FAN_CONTROL: now also R3.2
- new net: D2.2 (A), J3.2 (Pin_2), Q2.3 (D)
- new net: Q2.1 (G), R24.2, R3.1, TP5.1
Other:
- note added: "FAN CONTROL"
- note added: "Voltage_IN: Voltage for logic and MOSFET. Min: 4.5V Rec: 10V Max: 10V Current: 300-500mA"
- note removed: "Voltage_IN: Voltage for logic and MOSFET. Min: 4.5V Rec: 10V Max: 10V Current: 200-400mA"

Commit message: Intermediate commit, pre-update to new kicad
Parts:
- added D3: LED, LED_THT:LED_D5.0mm_Horizontal_O1.27mm_Z3.0mm, symbol Device:LED
- added R25: 220, Resistor_SMD:R_1206_3216Metric_Pad1.30x1.75mm_HandSolder, symbol Device:R
Connections:
- net 5V: now also R25.2
- net GND: now also D3.1 (K)
- new net: D3.2 (A), R25.1
Other:
- note added: "Vf = 2.2v"
- moved on the sheet: A1, SW1, U1C, U2

Commit message: Fix for PCB v1 and more sourcecode
Parts:
- R8: value 100 -> 330
Connections:
- net GND: now also A1.29 (GND), A1.4 (GND)
Changed lines of the file:
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@@
   (junction (at 157.48 57.15) (diameter 0) (color 0 0 0 0)
   )
+  (junction (at 45.085 165.735) (diameter 0) (color 0 0 0 0)
+  )
   (junction (at 264.16 80.01) (diameter 0) (color 0 0 0 0)
   )
@@
     (stroke (width 0) (type default) (color 0 0 0 0))
   )
+  (wire (pts (xy 48.26 165.735) (xy 45.085 165.735))
+    (stroke (width 0) (type default) (color 0 0 0 0))
+  )
   (wire (pts (xy 146.05 57.15) (xy 151.13 57.15))
     (stroke (width 0) (type default) (color 0 0 0 0))
@@
     (stroke (width 0) (type default) (color 0 0 0 0))
   )
+  (wire (pts (xy 45.085 163.195) (xy 48.26 163.195))
+    (stroke (width 0) (type default) (color 0 0 0 0))
+  )
   (wire (pts (xy 195.58 69.85) (xy 195.58 73.66))
     (stroke (width 0) (type default) (color 0 0 0 0))
@@
     (stroke (width 0) (type default) (color 0 0 0 0))
   )
+  (wire (pts (xy 45.085 165.735) (xy 45.085 168.275))
+    (stroke (width 0) (type default) (color 0 0 0 0))
+  )
   (wire (pts (xy 126.365 69.85) (xy 117.475 69.85))
     (stroke (width 0) (type default) (color 0 0 0 0))
@@
     (stroke (width 0) (type default) (color 0 0 0 0))
   )
+  (wire (pts (xy 45.085 165.735) (xy 45.085 163.195))
+    (stroke (width 0) (type default) (color 0 0 0 0))
+  )
   (wire (pts (xy 33.02 158.75) (xy 33.02 161.29))
     (stroke (width 0) (type default) (color 0 0 0 0))
@@
     )
   )
-  (global_label "BUTTON_ROT" (shape output) (at 85.725 133.985 0) (fields_autoplaced)
+  (global_label "BUTTON_ROT" (shape input) (at 85.725 133.985 0) (fields_autoplaced)
     (effects (font (size 1.27 1.27)) (justify left))
-    (property "Intersheet References" "${INTERSHEET_REFS}" (id 0) (at 3.81 -2.54 0)
-      (effects (font (size 1.27 1.27)) hide)
+    (property "Intersheet References" "${INTERSHEET_REFS}" (id 0) (at 99.7816 133.9056 0)
+      (effects (font (size 1.27 1.27)) (justify left) hide)
     )
   )
-  (global_label "BUTTON_OK" (shape output) (at 85.725 128.905 0) (fields_autoplaced)
+  (global_label "BUTTON_OK" (shape input) (at 85.725 128.905 0) (fields_autoplaced)
     (effects (font (size 1.27 1.27)) (justify left))
-    (property "Intersheet References" "${INTERSHEET_REFS}" (id 0) (at 3.81 -2.54 0)
-      (effects (font (size 1.27 1.27)) hide)
+    (property "Intersheet References" "${INTERSHEET_REFS}" (id 0) (at 98.814 128.8256 0)
+      (effects (font (size 1.27 1.27)) (justify left) hide)
     )
   )
@@
     )
   )
-  (global_label "BUTTON_BACK" (shape output) (at 85.725 131.445 0) (fields_autoplaced)
+  (global_label "BUTTON_BACK" (shape input) (at 85.725 131.445 0) (fields_autoplaced)
     (effects (font (size 1.27 1.27)) (justify left))
-    (property "Intersheet References" "${INTERSHEET_REFS}" (id 0) (at 3.81 -2.54 0)
-      (effects (font (size 1.27 1.27)) hide)
+    (property "Intersheet References" "${INTERSHEET_REFS}" (id 0) (at 101.1121 131.3656 0)
+      (effects (font (size 1.27 1.27)) (justify left) hide)
     )
   )
@@
       (effects (font (size 1.27 1.27)) (justify left))
     )
-    (property "Value" "100" (id 1) (at 158.75 36.83 90)
+    (property "Value" "330" (id 1) (at 158.75 36.83 90)
       (effects (font (size 1.27 1.27)) (justify left))
     )
@@
     (pin "1")
   )
+  (symbol (lib_id "power:GND") (at 45.085 168.275 0) (unit 1)
+    (in_bom yes) (on_board yes)
+    (property "Reference" "#PWR?" (id 0) (at 45.085 174.625 0)
+      (effects (font (size 1.27 1.27)) hide)
+    )
+    (property "Value" "GND" (id 1) (at 45.212 172.6692 0))
+    (property "Footprint" "" (id 2) (at 45.085 168.275 0)
+      (effects (font (size 1.27 1.27)) hide)
+    )
+    (property "Datasheet" "" (id 3) (at 45.085 168.275 0)
+      (effects (font (size 1.27 1.27)) hide)
+    )
+    (pin "1")
+  )
   (symbol (lib_id "Device:LED") (at 33.02 154.94 90) (unit 1)
     (in_bom yes) (on_board yes) (fields_autoplaced)
@@
       (reference "#PWR0102") (unit 1) (value "GND") (footprint "")
     )
+    (path "/5f253ba5-bbda-4c32-8fe5-5d3332a5b885"
+      (reference "#PWR?") (unit 1) (value "GND") (footprint "")
+    )
     (path "/00000000-0000-0000-0000-00006165dab4"
       (reference "A1") (unit 1) (value "Arduino_Nano") (footprint "Arduinos:arduino_nano")
@@
     )
     (path "/00000000-0000-0000-0000-00006037d4fe"
-      (reference "R8") (unit 1) (value "100") (footprint "Resistor_SMD:R_1206_3216Metric_Pad1.30x1.75mm_HandSolder")
+      (reference "R8") (unit 1) (value "330") (footprint "Resistor_SMD:R_1206_3216Metric_Pad1.30x1.75mm_HandSolder")
     )
     (path "/00000000-0000-0000-0000-00006036e71b"

Commit message: Version stable
Parts:
- removed R22: 2k2, Resistor_SMD:R_1206_3216Metric_Pad1.30x1.75mm_HandSolder, symbol Device:R
- R21: value 330 -> 1k
- renumbered R23 to R22
Connections:
- net at R22.2, U4.2 (REF): now also R21.1
Other:
- note added: "2.31"
- note added: "9.87"
- note added: "Analog_REF: Vref = (1+ R21/R22)*2.5 R21 = 1k R22 = 1k5 V = 4.16"
- note added: "Gain: ( (R2 +Pot)/R4 + 1 ) Adjust to have output: 0.0 - 4.16 V"
- note removed: "Analog_REF: V = 4.0"
- note removed: "Gain: ( (R2 +Pot)/R4 + 1 ) Adjust to have output: 0.0 - 4.0 V"
- moved on the sheet: R18, R21, R22, TP4, U4
